File: kicad/gen2-jtag-adapter.kicad_pcb (KiCad board)
At the start: 2 copper layers, 20.5 x 30.5 mm, 15 parts, among them J1 FTSH-105-01-F-DV-K, U1 PHOTON, U2 PARTICLE_LOGO_9MM

Commit message: updated silkscreen, v1.1
Other:
- board text added: "3V3"
- board text added: "v1.1"
- board text removed: "RST"
